File: logger/hardware/kicad/accord-logger.kicad_sch (KiCad schematic)
At the start: 91 parts, among them J1 Power 2-way, J2 Cluster harness 8-way, J3 Bus / expansion (unpopulated), J4 Service 4-way, J5 SD breakout 6-way, Q1 IRF4905PbF, Q2 2N3904, Q3 2N3904, U1 RaspberryPi_Pico_W, U2 PC817, U3 LM2678T-5.0, X1 SIGNAL_ISOLATION (required), X2 SIGNAL_ISOLATION (under revie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, X3 SIGNAL_ISOLATION (under revie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, X4 SIGNAL_ISOLATION (under revie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, X5 SIGNAL_ISOLATION (under revie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, X6 IGN_QUALIFICATION, X7 VEHICLE_PROTECTION, X8 MAX_ON

Commit message: LRA-12: resolve all eight placeholders into a routable design
Completes the LRA-06 capture into a complete electrical design the owner can
place and route on 80 x 120 mm. Every populated part carries a checked
footprint, ERC is clean at --severity-all, and no placeholder remains.

X7, the entry voltage envelope, is one forced chain rather than a menu. The
only P-FET the record found with a hot zero-gate leakage maximum that fits the
200 uA switch allocation is the IPD50P04P4L-11 at 70 uA/125 C, where the
IRF4905 screens 250 uA and cannot. That part is rated -40 V, so the clamp has
to hold below 40 V, which rules out the inherited 1.5KE30A at 41.4 V - the
same 41.4 V that already exceeded QI/QH VCEO and the LM2678 ceiling. The
1.5KE20A clamps at 27.7 V, 29.20 V at 85 C from its own 0.090 %/K
coefficient, leaving 10.8 V to every 40 V part. That still misses the 28 V
protected-rail target, so the A5 regulator gets its own second stage: 330 R
and a BZX55C22 hold P_AON at 25.70 V worst case, 4.30 V inside TPS709's 30 V.
The <=28 V criterion is now measured at TP_PAON, not at P12. Sustained P12 is
declared <=17.1 V and a 24 V jump start with the board connected is an
excluded exposure, because no clamp of this family both stands off 24 V and
limits to 28 V; the two alternatives are costed for review.

X1 implements the ASSR-601JV with a GPIO enable in series with a hardware
PGOOD permission, because BAD does not necessarily remove B5 - the original
design gates only QH and QI can hold power with ignition present, so a rail
argument could not carry fail-open. R_ISO is 270 R, not 330 R: 330 R put the
worst-case LED current at 8.64 mA, below the 10 mA the 4 ms turn-on maximum is
specified at, which would have left turn-on unspecified. The footprint is a
12-pad local variant built from the manufacturer land pattern, with pin 3
asserted unconnected and the absent pins 11-14 left clear.

X2-X5 are a decided bypass with a nine-state reachable-state table. All four
are ignition-f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
Parts:
- removed C4: 10-100uF, Capacitor_THT:CP_Radial_D6.3mm_P2.50mm, symbol Device:C_Polarized
- removed C6: 100uF/50V, Capacitor_THT:CP_Radial_D10.0mm_P5.00mm, symbol Device:C_Polarized
- removed C8: 10nF/50V, Capacitor_THT:C_Disc_D5.0mm_W2.5mm_P5.00mm, symbol Device:C
- removed D108: 1N5819, Diode_THT:D_DO-41_SOD81_P7.62mm_Horizontal, symbol Diode:1N5819
- removed D109: 1N4148, Diode_THT:D_DO-35_SOD27_P7.62mm_Horizontal, symbol Diode:1N4148
- removed D110, D113: SB360-E3/54, Diode_THT:D_DO-201AD_P12.70mm_Horizontal, symbol Device:D_Schottky
- removed D111: 1.5KE30A-E3/54, Diode_THT:D_DO-201AD_P12.70mm_Horizontal, symbol Device:D_TVS
- removed D112: BZX55C12, Diode_THT:D_DO-35_SOD27_P7.62mm_Horizontal, symbol Device:D_Zener
- removed D114: 1N4004-E3/54, Diode_THT:D_DO-41_SOD81_P7.62mm_Horizontal, symbol Diode:1N4004
- removed F2: 1A, Fuse:Fuseholder_Clip-5x20mm_Bel_FC-203-22_Lateral_P17.80x5.00mm_D1.17mm_Horizontal, symbol Device:Fuse
- removed J3: Bus / expansion (unpopulated), Connector_PinHeader_2.54mm:PinHeader_1x06_P2.54mm_Vertical, symbol Connector_Generic:Conn_01x06
- removed J4: Service 4-way, Connector_PinHeader_2.54mm:PinHeader_1x04_P2.54mm_Vertical, symbol Connector_Generic:Conn_01x04
- removed JP2: RUN reset link, Connector_PinHeader_2.54mm:PinHeader_1x02_P2.54mm_Vertical, symbol Jumper:Jumper_2_Open
- removed Q1: IRF4905PbF, Package_TO_SOT_THT:TO-220-3_Vertical, symbol Transistor_FET:IRF4905
- removed Q2, Q3: 2N3904, Package_TO_SOT_THT:TO-92_Inline, symbol Transistor_BJT:2N3904
- removed U3: LM2678T-5.0, Package_TO_SOT_THT:TO-220-7_P2.54x3.7mm_StaggerEven_Lead3.8mm_Vertical, symbol Custom:LM2678T-5.0
- removed X1: SIGNAL_ISOLATION (required), symbol Custom:PLACEHOLDER_SIGNAL_ISO_REQ
- removed X2, X3, X4, X5: SIGNAL_ISOLATION (under review), symbol Custom:PLACEHOLDER_SIGNAL_ISO_REVIEW
- removed X6: IGN_QUALIFICATION, symbol Custom:PLACEHOLDER_IGN_QUAL
- removed X7: VEHICLE_PROTECTION, symbol Custom:PLACEHOLDER_VEHICLE_PROT
- removed X8: MAX_ON, symbol Custom:PLACEHOLDER_MAX_ON
- added C11: 100nF/63V, Capacitor_THT:C_Disc_D5.0mm_W2.5mm_P5.00mm, symbol Device:C
- added C12: 10nF/50V, Capacitor_THT:C_Disc_D5.0mm_W2.5mm_P5.00mm, symbol Device:C
- added C13: 100nF/50V, Capacitor_THT:C_Disc_D5.0mm_W2.5mm_P5.00mm, symbol Device:C
- added C14: 1000uF/16V, Capacitor_THT:CP_Radial_D10.0mm_P5.00mm, symbol Device:C_Polarized
- added C15: 33uF/16V, Capacitor_Tantalum_SMD:CP_EIA-7343-31_Kemet-D_HandSolder, symbol Device:C_Polarized
- added C16: 10nF, Capacitor_THT:C_Disc_D5.0mm_W2.5mm_P5.00mm, symbol Device:C
- added C17, C18, C19, C20, C21, C22, C23: 100nF, Capacitor_THT:C_Disc_D5.0mm_W2.5mm_P5.00mm, symbol Device:C
- added C4, C6: 4.7uF/50V, Capacitor_SMD:C_1210_3225Metric_Pad1.33x2.70mm_HandSolder, symbol Device:C
- added C8: 47uF/16V, Capacitor_THT:CP_Radial_D6.3mm_P2.50mm, symbol Device:C_Polarized
- added D108, D113: 1.5KE20A-E3/54, Diode_THT:D_DO-201AD_P5.08mm_Vertical_KathodeUp, symbol Diode:1.5KExxA
- added D109: 1N5819, Diode_THT:D_DO-41_SOD81_P5.08mm_Vertical_AnodeUp, symbol Diode:1N5819
- added D110: 1N4148, Diode_THT:D_DO-35_SOD27_P2.54mm_Vertical_AnodeUp, symbol Diode:1N4148
- added D111: BZX55C22, Diode_THT:D_DO-35_SOD27_P2.54mm_Vertical_KathodeUp, symbol Device:D_Zener
- added D112, D115: SB360-E3/54, Diode_THT:D_DO-201AD_P5.08mm_Vertical_AnodeUp, symbol Device:D_Schottky
- added D114: BZX55C10, Diode_THT:D_DO-35_SOD27_P2.54mm_Vertical_KathodeUp, symbol Device:D_Zener
- added D116: 1N4004-E3/54, Diode_THT:D_DO-41_SOD81_P5.08mm_Vertical_KathodeUp, symbol Diode:1N4004
- added J3: Expansion 8-way (DNP bus), Connector_PinHeader_2.54mm:PinHeader_1x08_P2.54mm_Vertical, symbol Connector_Generic:Conn_01x08
- added J4: Reset RUN-GND, Connector_PinHeader_2.54mm:PinHeader_1x02_P2.54mm_Vertical, symbol Connector_Generic:Conn_01x02
- added Q1, Q6, Q7, Q9: 2N3904, Package_TO_SOT_THT:TO-92_Inline, symbol Transistor_BJT:2N3904
- added Q2, Q3, Q4, Q8: BSS138P, Package_TO_SOT_SMD:SOT-23, symbol Transistor_FET:BSS138
- added Q5: IPD50P04P4L-11, Package_TO_SOT_SMD:TO-252-3_TabPin2, symbol Transistor_FET:Q_PMOS_GDS
- added R24, R26, R29, R37, R38, R42: 1k, Resistor_THT:R_Axial_DIN0207_L6.3mm_D2.5mm_P5.08mm_Vertical, symbol Device:R
- added R25, R27, R34, R35, R41, R43, R45, R46: 100k, Resistor_THT:R_Axial_DIN0207_L6.3mm_D2.5mm_P5.08mm_Vertical, symbol Device:R
- added R28, R44: 47k, Resistor_THT:R_Axial_DIN0207_L6.3mm_D2.5mm_P5.08mm_Vertical, symbol Device:R
- added R30, R31, R36: 10k, Resistor_THT:R_Axial_DIN0207_L6.3mm_D2.5mm_P5.08mm_Vertical, symbol Device:R
- added R32: 1k, Resistor_THT:R_Axial_DIN0414_L11.9mm_D4.5mm_P5.08mm_Vertical, symbol Device:R
- added R33: 2.2k, Resistor_THT:R_Axial_DIN0207_L6.3mm_D2.5mm_P5.08mm_Vertical, symbol Device:R
- added R39, R40: 0R, Resistor_THT:R_Axial_DIN0207_L6.3mm_D2.5mm_P5.08mm_Vertical, symbol Device:R
- added TP21, TP22, TP23, TP24, TP25: TestPoint, TestPoint:TestPoint_Loop_D2.50mm_Drill1.0mm, symbol Connector:TestPoint
- added U10: CD74HC4060E, Package_DIP:DIP-16_W7.62mm, symbol Custom:CD74HC4060
- added U11: CD74HC4020E, Package_DIP:DIP-16_W7.62mm, symbol Custom:CD74HC4020
- added U12: CD4011BE, Package_DIP:DIP-14_W7.62mm, symbol Custom:CD4011B
- added U13: CD4071BE, Package_DIP:DIP-14_W7.62mm, symbol Custom:CD4071B
- added U14: CD4093BE, Package_DIP:DIP-14_W7.62mm, symbol Custom:CD4093B
- added U3: ASSR-601JV, accord-logger:ASSR-601Jx_SO-16-12Lead_11.634x10.363mm_P1.27mm, symbol Custom:ASSR-601JV
- added U4: TPS70950QDBVRQ1, Package_TO_SOT_SMD:SOT-23-5_HandSoldering, symbol Custom:TPS70950-Q1_DBV
- added U5: TPS3839K50DBZR, Package_TO_SOT_SMD:SOT-23, symbol Power_Supervisor:TPS3839DBZ
- added U6: LM2678T-5.0, Package_TO_SOT_THT:TO-220-7_P2.54x3.7mm_StaggerEven_Lead3.8mm_Vertical, symbol Custom:LM2678T-5.0
- added U7: OV-7604-C7-32.768KHZ-20PPM-TA-QC, accord-logger:Oscillator_SMD_MicroCrystal_OV-7604-C7_SON-4_3.2x1.5mm, symbol Custom:OV-7604-C7
- added U8: 74AHC1G17GV, Package_TO_SOT_SMD:SOT-353_SC-70-5_Handsoldering, symbol 74xGxx:74LVC1G17
- added U9: SN74LVC1G97DBVR, Package_TO_SOT_SMD:SOT-23-6_Handsoldering, symbol 74xGxx:74LVC1G97
- C10: value 820uF/16V -> 100uF/50V; footprint Capacitor_THT:CP_Radial_D12.5mm_P5.00mm -> Capacitor_THT:CP_Radial_D8.0mm_P3.50mm; MPN (none) -> Panasonic EEUFR1H101; Source DESIGN.md S3 -> COMPONENT_MARGIN_CLOSURE S1 / BOM_DELTA.csv; Source_designator COUT -> CIN; Status PART_SELECTION_OPEN -> CONDITIONAL
- C3: value 100nF -> 1uF; footprint Capacitor_THT:C_Disc_D5.0mm_W2.5mm_P5.00mm -> Capacitor_THT:C_Rect_L7.2mm_W2.5mm_P5.00mm_FKS2_FKP2_MKS2_MKP2; Source AS_BUILT S2 row 7 / S3.4 -> CUTOFF_MARGIN_REVIEW S2; Source_designator C_IGN -> CQUAL; Status VERIFY_OR_SOURCE -> PART_SELECTION_OPEN
- C5: value 100nF/63V -> 4.7uF/50V; footprint Capacitor_THT:C_Disc_D5.0mm_W2.5mm_P5.00mm -> Capacitor_SMD:C_1210_3225Metric_Pad1.33x2.70mm_HandSolder; MPN (none) -> Murata GRM32ER71H475KA88L; Source DESIGN.md S3 -> COMPONENT_MARGIN_CLOSURE S1 / BOM_DELTA.csv; Source_designator C0 -> C_A5A; Status VERIFY_OR_SOURCE -> CONDITIONAL
- C7: value 100nF/63V -> 100nF; Source DESIGN.md S3 -> CUTOFF_MARGIN_REVIEW S2; Source_designator CIB -> C_USUP
- C9: value 100nF/50V -> 100nF/63V; Source_designator COB -> C0
- D101, D102, D103, D104, D105, D106, D107: footprint Diode_THT:D_DO-41_SOD81_P7.62mm_Horizontal -> Diode_THT:D_DO-41_SOD81_P5.08mm_Vertical_AnodeUp
- F1: value 100mA -> 1A; Source DESIGN.md S3 / AS_BUILT S2 row 6 -> DESIGN.md S3 / LAYOUT_CLOSURE S3; Source_designator FIGN -> (none)
- J1: footprint (none) -> Connector_Molex:Molex_Mini-Fit_Jr_5569-02A2_2x01_P4.20mm_Horizontal; MPN (none) -> Molex 39-30-1020 (5569-02A2), 2 circuit right-angle header; Source REV_A_INTERFACES S5.1 / DESIGN.md S3 -> REV_A_INTERFACES S5.1 / LAYOUT_CLOSURE S6; Status PART_SELECTION_OPEN -> SELECTED
- J2: footprint (none) -> Connector_Molex:Molex_Mini-Fit_Jr_5569-08A2_2x04_P4.20mm_Horizontal; MPN (none) -> Molex 39-30-1080 (5569-08A2), 8 circuit right-angle header; Source REV_A_INTERFACES S5.1 -> REV_A_INTERFACES S5.1 / LAYOUT_CLOSURE S6; Status PART_SELECTION_OPEN -> SELECTED
- L1: Source DESIGN.md S3 -> DESIGN.md S3 / D-POWER-03 consequence 4
- R1, R10, R11, R12, R2, R3, R4, R5, R6, R7, R8, R9: footprint Resistor_THT:R_Axial_DIN0207_L6.3mm_D2.5mm_P7.62mm_Horizontal -> Resistor_THT:R_Axial_DIN0207_L6.3mm_D2.5mm_P5.08mm_Vertical
- R13: footprint Resistor_THT:R_Axial_DIN0414_L11.9mm_D4.5mm_P15.24mm_Horizontal -> Resistor_THT:R_Axial_DIN0414_L11.9mm_D4.5mm_P5.08mm_Vertical
- R14: value 10k -> 47k; footprint Resistor_THT:R_Axial_DIN0207_L6.3mm_D2.5mm_P7.62mm_Horizontal -> Resistor_THT:R_Axial_DIN0207_L6.3mm_D2.5mm_P5.08mm_Vertical; Source REV_A_INTERFACES S1 / DESIGN.md S3 -> CUTOFF_MARGIN_REVIEW S2; Source_designator RIGN -> RIGNA; Status VERIFY_STOCK -> VERIFY_OR_SOURCE
- R15: value 47k -> 220k; footprint Resistor_THT:R_Axial_DIN0207_L6.3mm_D2.5mm_P7.62mm_Horizontal -> Resistor_THT:R_Axial_DIN0207_L6.3mm_D2.5mm_P5.08mm_Vertical; Source REV_A_INTERFACES D2 / DESIGN.md S3 -> CUTOFF_MARGIN_REVIEW S2; Source_designator RPD -> RRC; Status VERIFY_STOCK -> VERIFY_OR_SOURCE
- R16: value 1k -> 22k; footprint Resistor_THT:R_Axial_DIN0207_L6.3mm_D2.5mm_P7.62mm_Horizontal -> Resistor_THT:R_Axial_DIN0207_L6.3mm_D2.5mm_P5.08mm_Vertical; Source DESIGN.md S3 -> CUTOFF_MARGIN_REVIEW S2; Source_designator RH -> R_RSTB
- R17: footprint Resistor_THT:R_Axial_DIN0207_L6.3mm_D2.5mm_P7.62mm_Horizontal -> Resistor_THT:R_Axial_DIN0207_L6.3mm_D2.5mm_P5.08mm_Vertical; Source DESIGN.md S3 -> CUTOFF_MARGIN_REVIEW S2; Source_designator RGS -> R_RSTPD
- R18: value 1k -> 4.7k; footprint Resistor_THT:R_Axial_DIN0414_L11.9mm_D4.5mm_P15.24mm_Horizontal -> Resistor_THT:R_Axial_DIN0207_L6.3mm_D2.5mm_P5.08mm_Vertical; Source DESIGN.md S3 -> CUTOFF_MARGIN_REVIEW S2; Source_designator RG -> R_RSTC
- R19: value 2.2k -> 1k; footprint Resistor_THT:R_Axial_DIN0207_L6.3mm_D2.5mm_P7.62mm_Horizontal -> Resistor_THT:R_Axial_DIN0207_L6.3mm_D2.5mm_P5.08mm_Vertical; Source DESIGN.md S3 -> CUTOFF_MARGIN_REVIEW S2; Source_designator RI -> R_REPG
- R20: footprint Resistor_THT:R_Axial_DIN0207_L6.3mm_D2.5mm_P7.62mm_Horizontal -> Resistor_THT:R_Axial_DIN0207_L6.3mm_D2.5mm_P5.08mm_Vertical; Source DESIGN.md S3 -> CUTOFF_MARGIN_REVIEW S2; Source_designator RBI -> R_REPPD
- R21: value 100k -> 10k; footprint Resistor_THT:R_Axial_DIN0207_L6.3mm_D2.5mm_P7.62mm_Horizontal -> Resistor_THT:R_Axial_DIN0207_L6.3mm_D2.5mm_P5.08mm_Vertical; Source DESIGN.md S3 -> REV_A_INTERFACES S1 / DESIGN.md S3; Source_designator RBH -> RIGN
- R22: value 10k -> 330R; footprint Resistor_THT:R_Axial_DIN0207_L6.3mm_D2.5mm_P7.62mm_Horizontal -> Resistor_THT:R_Axial_DIN0207_L6.3mm_D2.5mm_P5.08mm_Vertical; Source DESIGN.md S3 -> LAYOUT_CLOSURE S3; Source_designator RBIN -> R_AON; Status VERIFY_STOCK -> SELECTED
- R23: value 1k -> 270R; footprint Resistor_THT:R_Axial_DIN0207_L6.3mm_D2.5mm_P7.62mm_Horizontal -> Resistor_THT:R_Axial_DIN0207_L6.3mm_D2.5mm_P5.08mm_Vertical; Source DESIGN.md S3 -> LAYOUT_CLOSURE S4; Source_designator RB5 -> R_ISO; Status VERIFY_STOCK -> SELECTED
- TP10: Source_designator TP_QUALN -> TP_VCLK
- TP11: Source_designator TP_ARM -> TP_QUALN
- TP12: Source_designator TP_EXPIRED -> TP_IGNRC
- TP13: Source_designator TP_PGOOD -> TP_IGNQ
- TP14: Source_designator TP_HOLDN -> TP_CLK32
- TP15: Source_designator TP_HOLD -> TP_ARM
- TP16: Source_designator TP_GND_BUCK -> TP_EXPIRED
- TP17: Source_designator TP_GND_PICO -> TP_PGOOD
- TP18: Source_designator TP_GND_HARNESS -> TP_HOLDN
- TP19: Source_designator TP_GP11 -> TP_HOLD
- TP20: Source_designator TP_GP12 -> TP_ISOEN
- TP8: Source_designator TP_A5 -> TP_PAON
- TP9: Source_designator TP_VCLK -> TP_A5
- U2: MPN Sharp PC817XNNSZ1B or qualified equiv -> Sharp PC817XNNSZ1B or qualified equivalent; Source AS_BUILT S2 rows 6-7 / S3.4 -> AS_BUILT S2 rows 6-7 / S3.4; CUTOFF_MARGIN_REVIEW S2
Connections:
- net B11_ISO is gone; now on net B11_TAP: R10.1
- net B1_ISO is gone; now on net B1_TAP: R3.1
- net C11_ISO is gone; now on net C11_TAP: R7.1
- net C14_ISO is gone; now on net C14_TAP: R5.1
- net IGN_FUSED is gone; now on net BATT_F: F1.2
- net A5: now also C5.1, C7.1, TP9.1, U2.4, C18.1, C19.1, C20.1, C21.1, C22.1, C23.1, C6.1, R38.1, R46.2, U10.16 (VDD), U11.16 (VDD), U12.14 (VDD), U13.14 (VDD), U14.14 (VDD), U14.2 (A2), U4.5 (OUT), U5.3 (VDD), U9.5 (VCC); no longer TP8.1
- net AGND: now also TP23.1; no longer TP18.1, U2.2
- net ARM: now also TP15.1, R42.1, U12.3 (AY), U12.6 (B2), U8.2, U9.6 (IN2); no longer TP11.1
- net B11_TAP: now also D108.1 (A1), D109.2 (A); no longer F1.1
- net B2_ISO: now also U3.10 (D2), U3.9 (D2)
- net B2_TAP: now also U3.15 (D1), U3.16 (D1)
- net B5: now also C13.1, C14.1, D116.2 (A), J3.1 (Pin_1), R37.1, U6.6 (FEEDBACK); no longer C10.1, C9.1
- net BATT_F: now also D112.2 (A)
- net BATT_IN: now also F1.1
- net BOOST: now also C12.2, U6.3 (BOOST)
- net EXPIRED: now also TP16.1, R39.2, R40.2, R41.1, U13.9 (C2); no longer TP12.1
- net GATE: now also D114.2 (A), Q5.1 (G), R31.2, R32.1; no longer R17.2, R18.1
- net HOLD_B: now also Q7.2 (B), R29.2, R35.1; no longer R16.2, R21.1
- net HOLD_JH: now also R29.1; no longer R16.1
- net HOLD_N: now also TP18.1, Q9.3 (C), R46.1, U13.13 (D2); no longer TP14.1
- net HOLD_RAW: now also TP19.1, R28.1, R44.1; no longer R15.1, TP15.1
- net IGN_B: now also Q6.2 (B), R33.2, R34.1; no longer R19.2, R20.1
- net IGN_LED_A: now also D110.1 (K)
- net IGN_POS: now also D109.1 (K), R33.1; no longer R19.1
- net P12: now also C9.1, R22.1, D112.1 (K), D113.1 (A1), D114.1 (K), Q5.3 (S), R31.1; no longer C5.1, R17.1
- net P3V3_SW: now also R21.1, C8.1, J3.3 (Pin_3); no longer R14.1
- net PGND: now also R14.2, R17.2, U2.2, C11.2, C13.2, C14.2, C15.2, C16.2, C17.2, C18.2, C19.2, C20.2, C21.2, C22.2, C23.2, C4.2, C6.2, C8.2, D108.2 (A2), D110.2 (A), D111.2 (A), D113.2 (A2), D115.2 (A), J3.2 (Pin_2), J3.8 (Pin_8), J4.2 (Pin_2), Q1.1 (E), Q2.2 (S), Q4.2 (S), Q6.1 (E), Q7.1 (E), Q9.1 (E), R25.2, R27.2, R28.2, R30.2, R34.2, R35.2, R36.2, R37.2, R41.2, R43.2, R45.2, TP21.1, TP22.1, U10.8 (VSS), U11.8 (VSS), U12.12 (D1), U12.13 (D2), U12.7 (VSS), U13.7 (VSS), U14.7 (VSS), U4.2 (GND), U5.1 (GND), U6.4 (GND), U7.2 (GND), U8.3 (GND), U9.1 (IN1), U9.2 (GND); no longer R15.2, R21.2, R22.2, R23.2, TP16.1, TP17.1, U2.3
- net PGOOD: now also TP17.1, R26.1, U14.5 (B1), U14.6 (B2), U5.2 (~{RESET}); no longer TP13.1
- net QUAL_N_REPORT: now also R21.2, TP11.1, Q2.3 (D); no longer R14.2, TP10.1
- net RUN: now also J4.1 (Pin_1)
- net SINK: now also Q6.3 (C), Q8.3 (D), R32.2; no longer R18.2
- net SPARE_GP11: now also TP24.1; no longer TP19.1
- net SPARE_GP12: now also TP25.1; no longer TP20.1
- net SW: now also C12.1, D115.1 (K), U6.1 (SWITCH)
- net VCLK: now also TP10.1, C15.1, C16.1, C17.1, R38.2, U7.4 (VDD), U8.5 (VCC); no longer TP9.1
- net VIN_SW: now also C10.1, C11.1, Q5.2 (D), R36.1, U6.2 (VIN); no longer C7.1, R22.1
- net VSYS: now also D116.1 (K)
- net ISO_EN: now reaches U1.10 (GPIO7)
- net ISO_EN: now also TP20.1, R24.1
- net UART1_TX: now reaches U1.11 (GPIO8)
- net UART1_TX: now also J3.4 (Pin_4)
- net UART1_RX: now reaches U1.12 (GPIO9)
- net UART1_RX: now also J3.5 (Pin_5)
- net BUS_DE: now reaches U1.14 (GPIO10)
- net BUS_DE: now also J3.6 (Pin_6), R30.1
- net SPARE_GP13: now reaches U1.17 (GPIO13)
- net SPARE_GP13: now also J3.7 (Pin_7)
- net IGN_N renamed IGN_RC
- net IGN_RC: now also R15.2, R18.2, TP12.1, U14.1 (A1); no longer U2.4
- new net ARM_G: Q8.1 (G), R42.2, R43.1
- new net ARM_RESET: U13.11 (DY), U14.8 (C1), U14.9 (C2)
- new net BAD: R16.1, U13.1 (A1), U13.8 (C1), U14.4 (BY)
- new net BASE_RESET: U11.11 (MR), U13.3 (AY), U13.5 (B1)
- new net CLK32: TP14.1, U10.11 (CLK), U9.4 (Y)
- new net CLKOE: U7.3 (CLKOE), U8.4
- new net CNT_Q13: R39.1, U11.2 (Q13)
- new net CNT_Q8: R40.1, U11.13 (Q8)
- new net COUNT1_RESET: U10.12 (MR), U13.4 (BY)
- new net FAULT_RESET: U13.10 (CY), U13.12 (D1)
- new net IGN_A: R14.1, R15.1, U2.3
- new net IGN_Q: R19.1, TP13.1, U12.10 (CY), U13.2 (A2), U14.12 (D1)
- new net ISO_EN_G: Q4.1 (G), R24.2, R25.1
- new net ISO_LED_A: R23.2, U3.4 (AN)
- new net ISO_LED_K: Q3.3 (D), U3.5 (CA)
- new net ISO_MID: Q3.2 (S), Q4.3 (D)
- new net ISO_PG_G: Q3.1 (G), R26.2, R27.1
- new net MON_B: Q9.2 (B), R44.2, R45.1
- new net NARM: U12.2 (A2), U12.4 (BY), U13.6 (B2)
- new net P_AON: C4.1, D111.1 (K), R22.2, TP8.1, U4.1 (IN)
- new net QH_C: Q7.3 (C), Q8.2 (S)
- new net QUAL_N: U12.8 (C1), U12.9 (C2), U14.3 (AY)
- new net REP_G: Q2.1 (G), R19.2, R20.1
- new net RESET_N: U12.5 (B1), U14.10 (CY), U14.13 (D2)
- new net RST_B: Q1.2 (B), R16.2, R17.1
- new net RST_C: Q1.3 (C), R18.1
- new net SET_N: U12.1 (A1), U14.11 (DY)
- new net UCLK_Q14: U10.3 (Q14), U11.10 (CLK)
- new net XO_OUT: U7.1 (CLKOUT), U9.3 (IN0)
- no-connect marks 27 -> 37
Other:
- note added: "Classified in full in LRA12_HANDOFF.md. In short: ORDER GATE ASSR-601JV availability (fallback AQY221N2S specified, strictly smaller, same keepout); exact fuse family and curve; capacitor approval-sheet bias/aging/IR data. BRING-UP A5 ground current below 100 uA load; hot leakage of QP, QI, QH, QMON, QS, QREPORT and the opto; clock startup and loaded ramps; opto ON/OFF endpoints; ASSR turn-on aga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"
- note added: "EXPANSION (DNP BUS) AND RESET - LRA-04 bounded provision"
- note added: "Five fitted cells, carried forward with no value changed (AS_BUILT S2). B2 is the only branch energized with the key out - 4.669 V open circuit, 4.140 V loaded, drawing 140.8 uA of which 109.2 uA was being back-fed into the unpowered 3V3 rail through a forward-biased clamp. It gets the series switch, upstream of the divider top as required. B1, C14, C11 and B11 are all ignition-fed and measured o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"
- note added: "GP0/GP1, GP14/GP15, GP20-GP22 and GP28 are deliberately unconnected. GP7 is now ISO_EN, the B2 isolation enable, confirmed free in S1. GP8/GP9 (UART1) and GP10 (tied DE//RE) go to the DNP expansion header, with GP13 offered there as a spare - offers, not reservations. ARM, EXPIRED, PGOOD and HOLD_N stay off the GPIOs: A5-domain test points only, and firmware has no ARM feedback in this revision. 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"
- note added: "GP6 HOLD_RAW with a 47k external pulldown and the JH MAINTENANCE link. Firmware latches it LOW before output enable; 4 mA drive, 2.6 V loaded qualification target. QS is the series interruption the independent timer uses: drain to SINK, source to the QH collector, body diode blocking the sink direction when off. QI remains wired straight to SINK, so raw ignition still overrides everything. QMON s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"
- note added: "HOLD driver and the cutoff path"
- note added: "IGNITION OPTO CELL, VEHICLE SIDE - AS_BUILT S3.4; LED return moved to PGND"
- note added: "INDEPENDENT CLOCK BLOCK - CUTOFF_MARGIN_REVIEW S1"
- note added: "Independent cutoff - what it does and does not cover"
- note added: "LRA-12 - what changed, and the one thing to read first"
- note added: "NOTES - LRA-12 electrical closure"
- note added: "Nominal 2048 s from qualified ignition loss, on its own always-on supply and its own clock. The Pico cannot refresh it with HOLD, resets, network traffic or watchdog servicing; releasing HOLD disarms it, and only a qualified ignition assertion can grant it again. Reset dominates set in the settled Boolean model. UCOUNT is reset by BAD OR IGN_Q and deliberately NOT by NARM, which would erase EXPIR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"
- note added: "ONBOARD SWITCHED POWER - power/DESIGN.md S3, deltas D7 and D13, X7 entry clamp resolved"
- note added: "Reuses the existing power candidate as DESIGN.md S3 lists it (D-POWER-02), with the reviewed deltas D7 and D13 and the LRA-02 component selections. The LM2678, its TVS role, bulk capacitors, boost cap, inductor value and both Schottky positions all have in-service precedent on the keyless board in this car (D-POWER-03); the logger adds QP, QI/QH, DZ, DOR, the A5 rail and MAX_ON. Rail nets: P12 al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"
- note added: "SD and expansion"
- note added: "SPI0 at 12 MHz on switched 3V3 only (GP16 MISO, GP17 CS, GP18 SCK, GP19 MOSI). D6 bulk is now a selected 47 uF: a 200 mA write spike for 1 ms inside 100 mV of droop needs 2 uF, so this is an order of margin without an oversized can. Any move of this module to a 5 V rail re-opens the MISO clearance gate of AS_BUILT S3.5. J3 is a passive expansion header for a DNP daughterboard. There is no transce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"
- note added: "TEST POINTS AND GROUND LOOPS - REV_A_INTERFACES S5.3, delta D8"
- note added: "Test points and ground loops"
- note added: "The fitted cell returned the ignition LED cathode to the B16 cluster conductor with nothing in series, putting 4.7-5.8 mA of signal- dependent current through the node both ADC channels reference, which REV_A_INTERFACES S4 says must never become a power return. D5 and that return cannot both stand. LRA-12 moves the cathode to PGND, the arrangement DESIGN.md S3 already specified. What B16 still ca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"
- note added: "The opto LED return - R06-REV-2 decided"
- note added: "The selected QP is the only P-channel switch the record found with a HOT zero-gate leakage maximum (70 uA at 125 C) that fits the 200 uA parked allocation; the IRF4905 screen is 250 uA and cannot. That part is rated -40 V VDS, so the entry clamp has to hold below 40 V, which rules out the inherited 1.5KE30A at 41.4 V - the same 41.4 V that already exceeded QI/QH VCEO and the LM2678 operating ceil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"
- note added: "The voltage envelope, which is one chain and not five choices"
- note added: "This is the LRA-06 capture with its eight electrical placeholders resolved. Every populated part now carries a checked footprint and no dashed NOT SELECTED body remains. The decisions, their calculations and the residual gates are in power/LAYOUT_CLOSURE.md and LRA12_HANDOFF.md; read those before changing anything here. X1 B2 series isolation -> ASSR-601JV + 2-FET enable X2-X5 other four branches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"
- note added: "Twenty-five test loops. Three separate ground loops follow the keyless pattern: buck, Pico and harness end, the last on the bonded B16/AGND sense node. J4 shorts RUN to GND for a reset without cutting power. TP_PAON is where the <=28 V protected-rail criterion is measured. TP_GATE against TP_P12 is where the QP -14 to +1 V gate acceptance band is measured. TP_CLK32 carries the clock frequency and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"
- note added: "VEHICLE INPUTS - AS_BUILT S2, ratios and clamps unchanged; B2 series isolation fitted, other four branches bypassed"
- note added: "Vehicle inputs: one switch, four justified bypasses"
- note added: "What is still open - none of it a layout blocker"
- note added: "X1 ENABLE: GPIO PLUS HARDWARE PGOOD PERMISSION - LAYOUT_CLOSURE S4"
- note added: "X6 RESOLVED: QUALIFIED IGNITION, A5 DOMAIN - CUTOFF_MARGIN_REVIEW S2"
- note added: "X7 SECOND STAGE: ALWAYS-ON A5 SUPPLY AND SUPERVISOR - CUTOFF_MARGIN_REVIEW S3 + LAYOUT_CLOSURE S3"
- note added: "X8 RESOLVED: INDEPENDENT MAXIMUM-ON CUTOFF, 2048 s - MAX_ON_CUTOFF"
- note removed: "Fitted cell (AS_BUILT S3.4): B11 -> 1N5819 -> measured 2.2k -> LED anode; LED cathode returns to B16 with nothing in series; collector to the report path, emitter to PGND, fitted 100 nF across the output. No input capacitor. DESIGN.md S3 instead returns the LED to PGND and uses 1k/1N4148 - this capture follows the fitted cell, per the packet. Q2 raises the consequence: the fitted return puts 4.7-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"
- note removed: "Five fitted cells, carried forward with no value changed (AS_BUILT S2). Digital divider bottoms return to PGND. Both ADC divider bottoms, their filter and clamp returns, J2.6 (the B16 cluster ground sense) and Pico AGND are ONE node, bonded at a single point (S4, delta D5, R06-REV-1). Layout must not create a second path to it. B16 must never become a power return - but the fitted opto LED return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"
- note removed: "GP0/GP1, GP7, GP8-GP10 and GP28 are deliberately unconnected (X markers). GP8-GP10 are offers to LRA-04, not reservations. ARM, EXPIRED, PGOOD and HOLD_N stay off the GPIOs: they are A5-domain test points only. GP11 and GP12 are brought to pads per S1. ADC_VREF, 3V3_EN and VBUS are unconnected as fitted; VBUS has no buck connection (DESIGN.md S3)."
- note removed: "GP6 HOLD_RAW with a 47k external pulldown and the JH maintenance link. Firmware latches it LOW before output enable; 4 mA drive, 2.6 V loaded qualification target. Open JH for USB maintenance - RBH stays fitted."
- note removed: "HOLD driver"
- note removed: "IGNITION OPTO CELL - AS_BUILT S3.4, delta D1"
- note removed: "Ignition opto cell"
- note removed: "Independent maximum-on timer plus latched HOLD-path inhibit: 32-40 min after IGN fall, non-retriggerable by HOLD, <=40 uA room allocation. Not designed and not in stock record; required before unattended use. Its A5 and VCLK rails and its ARM/EXPIRED/PGOOD/HOLD_N status nodes are captured so layout cannot lose them. A5 also supplies XQUAL. HOLD_N is NOT inserted into the HOLD path by this capture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"
- note removed: "J3 BUS / J4 SERVICE - REV_A_INTERFACES S5.1"
- note removed: "J3 bus and J4 service"
- note removed: "J3 is unpopulated with every pin unconnected: LRA-04 selected no bus and reserved no pin. Do not capture a transceiver here. J4 carries the RUN-to-GND reset pair. Its UART0 pins are present but unconnected (Q5). It must be power-off-safe: no externally powered pull-up into an off GPIO."
- note removed: "LRA-06 CAPTURE - NOT FROZEN, NOT ACCEPTED, NOT FOR FABRICATION. Placeholders D4 (five instances), J3, MAX_ON and VEHICLE_PROTECTION carry no selected part. Open questions Q1-Q7 are in validation/../CAPTURE_NOTES.md."
- note removed: "MAX_ON"
- note removed: "MAX_ON - power BOM row, not implemented in revision A"
- note removed: "NOTES"
- note removed: "ONBOARD SWITCHED POWER - power/DESIGN.md S3, deltas D7 and D13"
- note removed: "PLACEHOLDER (dashed, "?", NOT SELECTED) = a block LRA-06 captures but does not resolve. X1-X5 are delta D4: normally-open, power-off-safe isolation upstream of a divider top. Five positions, one per branch, in two states after the owner key-out measurement of October 29 (D-OFFSTATE-01): REQUIRED - B2 only, and on a back-feed path rather than only a drain. Four readings in one configuration fix it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"
- note removed: "Placeholders, and delta D4"
- note removed: "Reuses the existing 9527a14 power candidate exactly as DESIGN.md S3 lists it (D-POWER-02), with two reviewed deltas: D7 onboard switched supply and D13 the 1N4004 DOR. Rail nets: P12 always-on, VIN_SW switched, B5 buck output, VSYS through DOR, P3V3_SW from the Pico regulator. QP body diode is drain-to-source: it blocks P12 to VIN_SW when off but does not block reverse energy. For every diode, ch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"
- note removed: "SD"
- note removed: "SPI0 at 12 MHz on switched 3V3 only (GP16 MISO, GP17 CS, GP18 SCK, GP19 MOSI). D6 adds bulk at the SD supply: write spikes of 100-200 mA otherwise land directly on the Pico's shared ~300 mA regulator. Any move of this module to a 5 V rail re-opens the MISO clearance gate of AS_BUILT S3.5 and must not be done in layout."
- note removed: "TEST POINTS AND RESET - REV_A_INTERFACES S5.3, delta D8"
- note removed: "Test loops per S5.3, plus TP_GATE and TP_SW from the power BOM TP row. Three separate ground loops, following the keyless pattern: buck, Pico and harness end. JR shorts RUN to GND for a reset without cutting power. Current-sensitive nodes must be measurable without the instrument supplying the current being measured, and probes must be removable for the final leakage reading - a layout requiremen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"
- note removed: "Test points and reset"
- note removed: "VEHICLE INPUTS - AS_BUILT S2, ratios and clamps unchanged"
- note removed: "Vehicle inputs"
- title: Accord logger Rev A - schematic capture (LRA-06) -> Accord logger Rev A - complete electrical design for layout (LRA-12)

Commit message: LRA-12R: correct clamp rationale, A5 thermal screen and schematic identities
Verify SQD50P06-15L as a valid hot-specified 60 V alternative; retain the
lower entry clamp for the logger A5 stage and LM2678 operating margin.
Correct the overvoltage exclusion to include regulator overcharge.
Raise R_AON to 820 ohm and account for zener junction heating, lead
conditions and the actual 16 V leakage test point. Record the accepted
allocation redistribution without changing 100/500 uA totals.

Generate deterministic UUID5 identities and verify unchanged generation,
placement/reannotation stability and uniqueness. ERC JSON: zero; capture:
652/652; closure: 63/63; 141/141 footprints, 1.52x allowance. Original
return and attribution are preserved; no hardware or deployment action.

Agent-Session: logger-electrical
Codex-Session-ID: 01a18a47-2dc2-7aa3-a0d2-a4978e2b1ebc
Parts:
- R22: value 330R -> 820R; Source LAYOUT_CLOSURE S3 -> LAYOUT_CLOSURE S3 (LRA-12R); Status SELECTED -> CONDITIONAL
Other:
- note added: "Retain 1.5KE20A by choice, not because a 60 V low-leakage QP is absent. SQD50P06-15L has 50 uA max IDSS at 125 C and -60 V. The inherited 1.5KE30A screens 43.81 V at 85 C: 1.19 V below LM2678 absolute, 3.81 V above operating. It also requires a redesigned A5 clamp. Selected 1.5KE20A screens 29.20 V. R_AON is now 820R/1%; the BZX55C22 thermal screen requires leads <=85 C. See S3 for bounds. P_AON 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"
- note added: "Voltage envelope - LRA-12R decision"
- note removed: "The selected QP is the only P-channel switch the record found with a HOT zero-gate leakage maximum (70 uA at 125 C) that fits the 200 uA parked allocation; the IRF4905 screen is 250 uA and cannot. That part is rated -40 V VDS, so the entry clamp has to hold below 40 V, which rules out the inherited 1.5KE30A at 41.4 V - the same 41.4 V that already exceeded QI/QH VCEO and the LM2678 operating ceil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"
- note removed: "The voltage envelope, which is one chain and not five choices"

Commit message: LRA-12R REV-4: reuse onboard keyless RS-485 with selectable bias
Carry MAX3485, DIP-8 socket footprint, 0805 decoupling and axial
bias/termination footprints from the exported keyless source. Assign
GP8/9/10, retain tied enables and 10k pulldown, use directed 390 ohm
bias values, and ship bias and termination headers without shunts.
Trim J3 to GP13 and switched power; add owner-approved interim
four-position Mini-Fit Jr for A/B/PGND/NC. Connector consolidation
and placement are separate work.

Record conditional external-bus currents and bias backfeed outside
the ordinary parked allocation. Correct derived-symbol footprint
inheritance so MAX3485 matches its library without ERC exclusions.

Validation: ERC JSON zero at severity-all; capture 711/711; closure
67/67; 150/150 footprints, 1.42x allowance. Consecutive generation is
byte-identical; UUID regression passes and previous component UUIDs
are preserved. No hardware, firmware, deployment or keyless edits.

Agent-Session: logger-electrical
Codex-Session-ID: 01a18a47-2dc2-7aa3-a0d2-a4978e2b1ebc
Parts:
- added C24: 100nF, Capacitor_SMD:C_0805_2012Metric_Pad1.18x1.45mm_HandSolder, symbol Device:C
- added J6: RS-485 interim A/B/GND, Connector_Molex:Molex_Mini-Fit_Jr_5569-04A2_2x02_P4.20mm_Horizontal, symbol Connector_Generic:Conn_01x04
- added JP2: TERM default OPEN, Connector_PinHeader_2.54mm:PinHeader_1x02_P2.54mm_Vertical, symbol Jumper:Jumper_2_Open
- added JP3: BIAS HI default OPEN, Connector_PinHeader_2.54mm:PinHeader_1x02_P2.54mm_Vertical, symbol Jumper:Jumper_2_Open
- added JP4: BIAS LO default OPEN, Connector_PinHeader_2.54mm:PinHeader_1x02_P2.54mm_Vertical, symbol Jumper:Jumper_2_Open
- added R47, R48: 390R, Resistor_THT:R_Axial_DIN0207_L6.3mm_D2.5mm_P5.08mm_Vertical, symbol Device:R
- added R49: 120R, Resistor_THT:R_Axial_DIN0207_L6.3mm_D2.5mm_P5.08mm_Vertical, symbol Device:R
- added U15: MAX3485, Package_DIP:DIP-8_W7.62mm, symbol Interface_UART:MAX3485
- J3: value Expansion 8-way (DNP bus) -> Spare GP13 / switched power; footprint Connector_PinHeader_2.54mm:PinHeader_1x08_P2.54mm_Vertical -> Connector_PinHeader_2.54mm:PinHeader_1x04_P2.54mm_Vertical; symbol Connector_Generic:Conn_01x08 -> Connector_Generic:Conn_01x04; Source LRA04_REVIEW_2026-10-29 / communications/REV_A_PROVISION.md -> D-RS485-05 / communications/REV_A_PROVISION.md
Connections:
- net BUS_DE: now also U15.2 (~{RE}), U15.3 (DE); no longer J3.6 (Pin_6)
- net P3V3_SW: now also C24.1, JP3.1 (A), U15.8 (VCC)
- net PGND: now also C24.2, J6.3 (Pin_3), JP4.2 (B), U15.5 (GND); no longer J3.8 (Pin_8)
- net SPARE_GP13: now also J3.4 (Pin_4); no longer J3.7 (Pin_7)
- net UART1_RX: now also U15.1 (RO); no longer J3.5 (Pin_5)
- net UART1_TX: now also U15.4 (DI); no longer J3.4 (Pin_4)
- new net RS485_A: J6.1 (Pin_1), R47.2, R49.1, U15.6 (A)
- new net RS485_B: J6.2 (Pin_2), JP2.2 (B), R48.1, U15.7 (B)
- new net RS485_BIAS_HI: JP3.2 (B), R47.1
- new net RS485_BIAS_LO: JP4.1 (A), R48.2
- new net RS485_TERM: JP2.1 (A), R49.2
- no-connect marks 37 -> 38
Other:
- note added: "GP0/GP1, GP14/GP15, GP20-GP22 and GP28 are deliberately unconnected. GP7 is now ISO_EN, the B2 isolation enable, confirmed free in S1. GP8/GP9 (UART1) and GP10 (tied DE//RE) drive onboard RS-485. GP13 is offered on the trimmed J3 spare/power header. ARM, EXPIRED, PGOOD and HOLD_N stay off the GPIOs: A5-domain test points only, and firmware has no ARM feedback in this revision. GP11 and GP12 are b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"
- note added: "RS-485 - keyless circuit; bias and termination OPEN by default"
- note added: "SPARE GP13 / SWITCHED POWER AND RESET"
- note added: "SPI0 at 12 MHz on switched 3V3 only (GP16 MISO, GP17 CS, GP18 SCK, GP19 MOSI). D6 bulk is now a selected 47 uF: a 200 mA write spike for 1 ms inside 100 mV of droop needs 2 uF, so this is an order of margin without an oversized can. Any move of this module to a 5 V rail re-opens the MISO clearance gate of AS_BUILT S3.5. RS-485 reuses keyless MAX3485, DIP-8, tied DE//RE and 10k pulldown. 390R bias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"
- note removed: "EXPANSION (DNP BUS) AND RESET - LRA-04 bounded provision"
- note removed: "GP0/GP1, GP14/GP15, GP20-GP22 and GP28 are deliberately unconnected. GP7 is now ISO_EN, the B2 isolation enable, confirmed free in S1. GP8/GP9 (UART1) and GP10 (tied DE//RE) go to the DNP expansion header, with GP13 offered there as a spare - offers, not reservations. ARM, EXPIRED, PGOOD and HOLD_N stay off the GPIOs: A5-domain test points only, and firmware has no ARM feedback in this revision. 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"
- note removed: "SPI0 at 12 MHz on switched 3V3 only (GP16 MISO, GP17 CS, GP18 SCK, GP19 MOSI). D6 bulk is now a selected 47 uF: a 200 mA write spike for 1 ms inside 100 mV of droop needs 2 uF, so this is an order of margin without an oversized can. Any move of this module to a 5 V rail re-opens the MISO clearance gate of AS_BUILT S3.5. J3 is a passive expansion header for a DNP daughterboard. There is no transce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"
