File: logger/hardware/kicad/accord-logger.kicad_sch (KiCad schematic)
At the start: 150 parts, among them J1 Power 2-way, J2 Cluster harness 8-way, J3 Spare GP13 / switched power, J4 Reset RUN-GND, J5 SD breakout 6-way, J6 RS-485 interim A/B/GND, Q1 2N3904, Q2 BSS138P, Q3 BSS138P, Q4 BSS138P, Q5 IPD50P04P4L-11, Q6 2N3904, Q7 2N3904, Q8 BSS138P, Q9 2N3904, U1 RaspberryPi_Pico_W, U10 CD74HC4060E, U11 CD74HC4020E, U12 CD4011BE, U13 CD4071BE, U14 CD4093BE, U15 MAX3485, U2 PC817, U3 ASSR-601JV, U4 TPS70950QDBVRQ1, U5 TPS3839K50DBZR, U6 LM2678T-5.0, U7 OV-7604-C7-32.768KHZ-20PPM-TA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, U8 74AHC1G17GV, U9 SN74LVC1G97DBVR

Commit message: logger hardware: single 10-way J1 board connector; docs to current state
Owner decision D-CONN-06: the owner's in-stock Molex 39-30-1100
(Mini-Fit Jr. 5569-10A2) replaces the 2-way J1, the 8-way J2 and the
interim 4-way RS-485 J485. Cavities: 1 BATT_IN, 2 B11, 3 B1, 4 C11,
5 RS485_A, 6 PGND, 7 AGND/B16, 8 C14, 9 B2, 10 RS485_B. The footprint
geometry matches the owner's own CON_39301100 file.

check_capture.py asserts the full pin map, that J1 is the only harness
connector, and, from the installed footprint's pad positions, that
BATT_IN's physical neighbours are only PGND and the clamped B11 input
and that A/B are adjacent.

Results: ERC 0 at severity-all, 721/721 capture, UUID regression pass
(1448), closure 67 ok, 1.48x courtyard allowance, two generations
byte-identical. Refresh README, REV_A_CONTEXT, COMMANDS and STATUS, and
add dated supersession notes to LAYOUT_CLOSURE 6.3, REV_A_PROVISION,
CAPTURE_NOTES and LRA12_HANDOFF.

Claude-Session-ID: 42dd0e33-28b5-4936-847e-9c2e1d2488fa

Co-Authored-By: Claude Opus 5.5 <noreply@anthropic.com>
Parts:
- removed J2: Cluster harness 8-way, Connector_Molex:Molex_Mini-Fit_Jr_5569-08A2_2x04_P4.20mm_Horizontal, symbol Connector_Generic:Conn_01x08
- removed J6: RS-485 interim A/B/GND, Connector_Molex:Molex_Mini-Fit_Jr_5569-04A2_2x02_P4.20mm_Horizontal, symbol Connector_Generic:Conn_01x04
- J1: value Power 2-way -> Board connector 10-way; footprint Connector_Molex:Molex_Mini-Fit_Jr_5569-02A2_2x01_P4.20mm_Horizontal -> Connector_Molex:Molex_Mini-Fit_Jr_5569-10A2_2x05_P4.20mm_Horizontal; symbol Connector_Generic:Conn_01x02 -> Connector_Generic:Conn_01x10; MPN Molex 39-30-1020 (5569-02A2), 2 circuit right-angle header -> Molex 39-30-1100 (5569-10A2), 10 circuit right-angle header; Source REV_A_INTERFACES S5.1 / LAYOUT_CLOSURE S6 -> DECISIONS D-CONN-06
Connections:
- net AGND: now also J1.7 (Pin_7)
- net B11_TAP: now also J1.2 (Pin_2)
- net B1_TAP: now also J1.3 (Pin_3)
- net B2_TAP: now also J1.9 (Pin_9)
- net C11_TAP: now also J1.4 (Pin_4)
- net C14_TAP: now also J1.8 (Pin_8)
- net PGND: now also J1.6 (Pin_6); no longer J1.2 (Pin_2)
- net RS485_A: now also J1.5 (Pin_5)
- net RS485_B: now also J1.10 (Pin_10)
- no-connect marks 38 -> 35
