File: logger/hardware/kicad/accord-logger.kicad_sch (KiCad schematic)
At the start: 153 parts, among them J1 Board connector 14-way, J3 Spare GP13 / switched power, J4 Reset RUN-GND, J5 SD breakout 6-way, Q1 MMBT3904, Q2 BSS138P, Q3 BSS138P, Q4 BSS138P, Q5 IPD50P04P4L-11, Q6 2N3904, Q7 2N3904, Q8 BSS138P, Q9 MMBT3904, U1 RaspberryPi_Pico_W, U10 CD74HC4060M96, U11 CD74HC4020M96, U12 CD4011BM96, U13 CD4071BM96, U14 CD4093BM96, U15 MAX3485, U16 DS3231SN, U2 PC817, U3 ASSR-601JV, U4 TPS70950QDBVRQ1, U5 TPS3839K50DBZR, U6 LM2678T-5.0, U7 OV-7604-C7-32.768KHZ-20PPM-TA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, U8 74AHC1G17GV, U9 SN74LVC1G97DBVR

Commit message: schematic: through-hole resistors and 1N5819 from the inputs on (D-THT-15)
Owner: "here I want to start using
Resistor_THT:R_Axial_DIN0204_L3.6mm_D1.6mm_P5.08mm_Horizontal and 1N5819
not 1N5819HW". All 37 surface-mount resistors except the placed RTC
pull-ups move to DIN0204; the eight 1N5819HW (D101-D107, D109) go back to
1N5819 on DO-41 vertical P5.08, the footprint they had before D-SMD-09.
R22 R_AON's >= 0.15 W at 85 C is met by a derated 0.25 W DIN0204 (noted in
the BOM). Also carries the owner's in_tach step switch-on (three flags).

check_capture.py: the package checks now assert DIN0204 resistors (bar
the RTC pull-ups) and the DO-41 1N5819; DI's value is 1N5819. ERC 0;
full-netlist capture 782/782, netlist changed only in footprint and value
fields; closure 67/67; courtyard allowance 1.61x.

Claude-Session-ID: 42dd0e33-28b5-4936-847e-9c2e1d2488fa
Co-Authored-By: Claude Opus 5.5 <noreply@anthropic.com>
Parts:
- D101, D102, D103, D104, D105, D106, D107, D109: value 1N5819HW -> 1N5819; footprint Diode_SMD:D_SOD-123 -> Diode_THT:D_DO-41_SOD81_P5.08mm_Vertical_AnodeUp
- R1, R10, R22, R3, R39, R40, R5, R7: footprint Resistor_SMD:R_1206_3216Metric_Pad1.30x1.75mm_HandSolder -> Resistor_THT:R_Axial_DIN0204_L3.6mm_D1.6mm_P5.08mm_Horizontal
- R11, R12, R14, R15, R16, R17, R18, R19, R2, R20, R21, R23, R24, R25, R26, R27, R28, R29, R38, R4, R41, R42, R43, R44, R45, R46, R6, R8, R9: footprint Resistor_SMD:R_0805_2012Metric_Pad1.20x1.40mm_HandSolder -> Resistor_THT:R_Axial_DIN0204_L3.6mm_D1.6mm_P5.08mm_Horizontal
